File: hardware/tangADC.kicad_sch (KiCad schematic)
At the start: 52 parts, among them J1 screw, J2 Conn_01x12_Pin, J3 RJ-2410N, J4 Conn_01x04_Pin, J5 Conn_01x04_Pin, U1 AD9280ARS, U2 Tang_Nano_20K

Commit message: Carrier board v0.2: AIN bias, chip parts, ground vias, edge clearance
Design files only; v0.2 has not been manufactured.  The board as built is
tag v0.1, and hardware/jlcpcb/ still holds v0.1's production files.

- R2 22k -> 10k and a new R19, 47k from AIN to CLAMPIN: AIN gets a DC
  path, and CLAMPIN is 1.0 V instead of 0.625.
- C13 is an 0603 in place of the leaded disc under the module.
- FB1 and FB2 are 0805 chip beads (LCSC C1017, a JLCPCB Basic part).
  The leaded parts doubled as jumpers, so the GND link under FB1 is
  0.6 mm wide there and vias stand where the four holes were.
- GND vias beside U1's ground pins 1, 14 and 16..18.
- The top-edge GND track is 0.69 mm from the edge (was 0.22).
- Silkscreen: revision, Grove 5 V note, J1 polarity, test-point legend.
- Stale no-connect flags in the schematic put right (ERC 14 -> 6).

kicad-cli pcb drc --schematic-parity: nothing unconnected, no parity
error, no clearance error.  docs/pcb-respin.md 4.6 has the details.

Co-Authored-By: Claude Opus 5.5 <noreply@anthropic.com>
Parts:
- added R19: 47k, Resistor_SMD:R_0603_1608Metric, symbol Device:R_Small
- C13: footprint Capacitor_THT:C_Disc_D3.0mm_W2.0mm_P2.50mm -> Capacitor_SMD:C_0603_1608Metric_Pad1.08x0.95mm_HandSolder
- FB1, FB2: value FerriteBead -> 600R@100MHz; footprint Resistor_THT:R_Axial_DIN0204_L3.6mm_D1.6mm_P5.08mm_Horizontal -> Inductor_SMD:L_0805_2012Metric
- R2: value 22k -> 10k
Connections:
- net at C13.1, R3.1, TP1.1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: now also R19.1
- net at C12.1, R2.2, R4.1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: now also R19.2
- no-connect marks 17 -> 19
Changed lines of the file:
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@@
 	)
 	(junction
+		(at 115.57 54.61)
+		(diameter 0)
+		(color 0 0 0 0)
+	)
+	(junction
 		(at 69.85 87.63)
 		(diameter 0)
@@
 	)
 	(junction
+		(at 115.57 49.53)
+		(diameter 0)
+		(color 0 0 0 0)
+	)
+	(junction
 		(at 142.24 38.1)
 		(diameter 0)
@@
 	)
 	(no_connect
-		(at 86.36 135.89)
+		(at 86.36 140.97)
 	)
 	(no_connect
-		(at 50.8 143.51)
+		(at 143.51 146.05)
 	)
 	(no_connect
-		(at 86.36 171.45)
+		(at 50.8 143.51)
 	)
 	(no_connect
@@
 	)
 	(no_connect
-		(at 50.8 135.89)
+		(at 143.51 148.59)
 	)
 	(no_connect
@@
 	)
 	(no_connect
+		(at 86.36 143.51)
+	)
+	(no_connect
 		(at 50.8 153.67)
 	)
 	(no_connect
+		(at 50.8 163.83)
+	)
+	(no_connect
 		(at 86.36 148.59)
 	)
@@
 		(shape input)
 		(at 184.15 72.39 0)
-		(fields_autoplaced yes)
 		(effects
 			(font
@@
 		(shape input)
 		(at 93.98 54.61 180)
-		(fields_autoplaced yes)
 		(effects
 			(font
@@
 		(shape input)
 		(at 143.51 140.97 0)
-		(fields_autoplaced yes)
 		(effects
 			(font
@@
 		(shape input)
 		(at 162.56 62.23 0)
-		(fields_autoplaced yes)
 		(effects
 			(font
@@
 		(shape input)
 		(at 229.87 115.57 0)
-		(fields_autoplaced yes)
 		(effects
 			(font
@@
 		(shape input)
 		(at 50.8 140.97 180)
-		(fields_autoplaced yes)
 		(effects
 			(font
@@
 		(shape input)
 		(at 184.15 85.09 0)
-		(fields_autoplaced yes)
 		(effects
 			(font
@@
 		(shape input)
 		(at 118.11 64.77 180)
-		(fields_autoplaced yes)
 		(effects
 			(font
@@
 		(shape input)
 		(at 184.15 67.31 0)
-		(fields_autoplaced yes)
 		(effects
 			(font
@@
 		(shape input)
 		(at 184.15 74.93 0)
-		(fields_autoplaced yes)
 		(effects
 			(font
@@
 		(shape input)
 		(at 50.8 158.75 180)
-		(fields_autoplaced yes)
 		(effects
 			(font
@@
 		(shape input)
 		(at 43.18 173.99 180)
-		(fields_autoplaced yes)
 		(effects
 			(font
@@
 		(shape input)
 		(at 195.58 115.57 0)
-		(fields_autoplaced yes)
 		(effects
 			(font
@@
 		(shape input)
 		(at 50.8 151.13 180)
-		(fields_autoplaced yes)
 		(effects
 			(font
@@
 		(shape input)
 		(at 175.26 90.17 0)
-		(fields_autoplaced yes)
 		(effects
 			(font
@@
 		(shape input)
 		(at 118.11 74.93 180)
-		(fields_autoplaced yes)
 		(effects
 			(font
@@
 		(shape input)
 		(at 86.36 173.99 0)
-		(fields_autoplaced yes)
 		(effects
 			(font
@@
 		(shape input)
 		(at 102.87 158.75 0)
-		(fields_autoplaced yes)
 		(effects
 			(font
@@
 		(shape input)
 		(at 143.51 143.51 0)
-		(fields_autoplaced yes)
 		(effects
 			(font
@@
 		(shape input)
 		(at 184.15 69.85 0)
-		(fields_autoplaced yes)
 		(effects
 			(font
@@
 		(shape input)
 		(at 82.55 91.44 0)
-		(fields_autoplaced yes)
 		(effects
 			(font
@@
 		(shape input)
 		(at 102.87 153.67 0)
-		(fields_autoplaced yes)
 		(effects
 			(font
@@
 		(shape input)
 		(at 143.51 130.81 0)
-		(fields_autoplaced yes)
 		(effects
 			(font
@@
 		(shape input)
 		(at 86.36 135.89 0)
-		(fields_autoplaced yes)
 		(effects
 			(font
@@
 		(shape input)
 		(at 143.51 133.35 0)
-		(fields_autoplaced yes)
 		(effects
 			(font
@@
 		(shape input)
 		(at 195.58 118.11 0)
-		(fields_autoplaced yes)
 		(effects
 			(font
@@
 		(shape input)
 		(at 43.18 168.91 180)
-		(fields_autoplaced yes)
 		(effects
 			(font
@@
 		(shape input)
 		(at 50.8 130.81 180)
-		(fields_autoplaced yes)
 		(effects
 			(font
@@
 		(shape input)
 		(at 229.87 118.11 0)
-		(fields_autoplaced yes)
 		(effects
 			(font
@@
 		(shape input)
 		(at 111.76 83.82 270)
-		(fields_autoplaced yes)
 		(effects
 			(font
@@
 		(shape input)
 		(at 43.18 166.37 180)
-		(fields_autoplaced yes)
 		(effects
 			(font
@@
 		(shape input)
 		(at 143.51 135.89 0)
-		(fields_autoplaced yes)
 		(effects
 			(font
@@
 		(shape input)
 		(at 43.18 171.45 180)
-		(fields_autoplaced yes)
 		(effects
 			(font
@@
 		(shape input)
 		(at 171.45 49.53 0)
-		(fields_autoplaced yes)
 		(effects
 			(font
@@
 		(shape input)
 		(at 184.15 82.55 0)
-		(fields_autoplaced yes)
 		(effects
 			(font
@@
 		(shape input)
 		(at 184.15 77.47 0)
-		(fields_autoplaced yes)
 		(effects
 			(font
@@
 		(shape input)
 		(at 50.8 161.29 180)
-		(fields_autoplaced yes)
 		(effects
 			(font
@@
 		(shape input)
 		(at 50.8 148.59 180)
-		(fields_autoplaced yes)
 		(effects
 			(font
@@
 		(shape input)
 		(at 69.85 74.93 90)
-		(fields_autoplaced yes)
 		(effects
 			(font
@@
 		(shape input)
 		(at 203.2 50.8 0)
-		(fields_autoplaced yes)
 		(effects
 			(font
@@
 		(shape input)
 		(at 50.8 135.89 180)
-		(fields_autoplaced yes)
 		(effects
 			(font
@@
 		(shape input)
 		(at 86.36 171.45 0)
-		(fields_autoplaced yes)
 		(effects
 			(font
@@
 		(shape input)
 		(at 184.15 80.01 0)
-		(fields_autoplaced yes)
 		(effects
 			(font
@@
 		(shape input)
 		(at 50.8 133.35 180)
-		(fields_autoplaced yes)
 		(effects
 			(font
@@
 		(shape input)
 		(at 143.51 138.43 0)
-		(fields_autoplaced yes)
 		(effects
 			(font
@@
 			)
 		)
-		(property "Value" "FerriteBead"
+		(property "Value" "600R@100MHz"
 			(at 31.496 181.864 90)
 			(show_name no)
@@
 			)
 		)
-		(property "Footprint" "Resistor_THT:R_Axial_DIN0204_L3.6mm_D1.6mm_P5.08mm_Horizontal"
+		(property "Footprint" "Inductor_SMD:L_0805_2012Metric"
 			(at 34.29 178.308 90)
 			(hide yes)
@@
 	)
 	(symbol
+		(lib_id "Device:R_Small")
+		(at 115.57 52.07 0)
+		(mirror y)
+		(unit 1)
+		(body_style 1)
+		(exclude_from_sim no)
+		(in_bom yes)
+		(on_board yes)
+		(in_pos_files yes)
+		(dnp no)
+		(property "Reference" "R19"
+			(at 113.03 50.7999 0)
+			(show_name no)
+			(do_not_autoplace no)
+			(effects
+				(font
+					(size 1.27 1.27)
+				)
+				(justify left)
+			)
+		)
+		(property "Value" "47k"
+			(at 113.03 53.3399 0)
+			(show_name no)
+			(do_not_autoplace no)
+			(effects
+				(font
+					(size 1.27 1.27)
+				)
+				(justify left)
+			)
+		)
+		(property "Footprint" "Resistor_SMD:R_0603_1608Metric"
+			(at 115.57 52.07 0)
+			(hide yes)
+			(show_name no)
+			(do_not_autoplace no)
+			(effects
+				(font
+					(size 1.27 1.27)
+				)
+			)
+		)
+		(property "Datasheet" ""
+			(at 115.57 52.07 0)
+			(hide yes)
+			(show_name no)
+			(do_not_autoplace no)
+			(effects
+				(font
+					(size 1.27 1.27)
+				)
+			)
+		)
+		(property "Description" "Resistor, small symbol"
+			(at 115.57 52.07 0)
+			(hide yes)
+			(show_name no)
+			(do_not_autoplace no)
+			(effects
+				(font
+					(size 1.27 1.27)
+				)
+			)
+		)
+		(pin "1"
+		)
+		(pin "2"
+		)
+		(instances
+			(project "tangADC"
+				(path "/58c7d11b-3319-4019-804f-829ad77d6f01"
+					(reference "R19")
+					(unit 1)
+				)
+			)
+		)
+	)
+	(symbol
 		(lib_id "Device:R")
 		(at 170.18 74.93 270)
@@
 			)
 		)
-		(property "Value" "FerriteBead"
+		(property "Value" "600R@100MHz"
 			(at 102.108 175.514 90)
 			(show_name no)
@@
 			)
 		)
-		(property "Footprint" "Resistor_THT:R_Axial_DIN0204_L3.6mm_D1.6mm_P5.08mm_Horizontal"
+		(property "Footprint" "Inductor_SMD:L_0805_2012Metric"
 			(at 100.33 170.688 90)
 			(hide yes)
@@
 			)
 		)
-		(property "Footprint" "Capacitor_THT:C_Disc_D3.0mm_W2.0mm_P2.50mm"
+		(property "Footprint" "Capacitor_SMD:C_0603_1608Metric_Pad1.08x0.95mm_HandSolder"
 			(at 112.0648 41.91 0)
 			(hide yes)
@@
 			)
 		)
-		(property "Value" "22k"
+		(property "Value" "10k"
 			(at 97.536 56.642 90)
 			(show_name no)

Commit message: Board v0.2: no Extended parts, and the production files for it
Every part JLCPCB places is now from its Basic or Preferred library
(12 Basic, 1 Preferred); v0.1 had two Extended parts.

- C7: the 1 uF tantalum becomes a 1206 X7R ceramic (C1848) on the same
  pads.
- D1: PESD5V0U1BA in SOD-323 becomes an H5VL10B in DFN1006-2L
  (C7420372, footprint D_SOD-882), still bidirectional.  No fee-free
  bidirectional ESD part exists in SOD-323.
- BOM, CPL and Gerbers regenerated for v0.2, in the JLCPCB-tools
  plugin's layout; its project.db carries the same LCSC numbers.

The Gerbers come from kicad-cli.  The same commands run on the v0.1
board reproduce seven of the nine ordered layers and both drill files
byte for byte apart from the date; the other two differ by one pour
vertex and by the mask openings of the four mounting holes.

kicad-cli pcb drc --schematic-parity: nothing unconnected, no parity
error, no clearance error.  docs/pcb-respin.md 4.7 has the details.

Co-Authored-By: Claude Opus 5.5 <noreply@anthropic.com>
Parts:
- D1: value PESD5V0U1BA -> H5VL10B; footprint Diode_SMD:D_SOD-323 -> Diode_SMD:D_SOD-882
Changed lines of the file:
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@@
 			)
 		)
-		(property "Value" "PESD5V0U1BA"
+		(property "Value" "H5VL10B"
 			(at 62.992 63.754 0)
 			(show_name no)
@@
 			)
 		)
-		(property "Footprint" "Diode_SMD:D_SOD-323"
+		(property "Footprint" "Diode_SMD:D_SOD-882"
 			(at 62.23 57.15 0)
 			(hide yes)
@@
 		)
 	)
-	(embedded_fonts no)
 )
